File: devboard/glitcher.kicad_sch (KiCad schematic)
At the start: 79 parts, among them J1 USB_C_Receptacle_USB2.0, J2 Conn_01x02, J3 IN, J4 OUT, J5 Conn_01x02, Q1 DMN3300U, SW3 SW_Push, U1 RP2040, U3 W25Q128JVS, U5 AMS1117-3.3, U5 COS722SR, U6 MS9280, Y1 12MHz

Commit message: Added merged devboard
Connections:
- net at U1.15 (GPIO12): now also R21.2
- net at U1.16 (GPIO13): no longer R21.2
- no-connect marks 3 -> 4
