File: glitcher/glitcher.kicad_pcb (KiCad board)
At the start: 4 copper layers, 44.1 x 84.5 mm, 80 parts, among them J1 USB_C_Receptacle_USB2.0, J3 Conn_01x05, J4 Conn_01x05, J5 Conn_01x03, J6 Conn_01x05, J7 Conn_01x03, Q1 DMN3300U, U1 RP2040, U2 AMS1117-3.3, U3 W25Q128JVS, U4 AMS1117-3.3, U5 COS722SR, U6 MS9280, Y1 12MHz

Commit message: Added silkscreen
Other:
- board text added: "ADC ->"
- board text added: "GLITCHER"
Changed lines of the file:
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@@
   (gr_curve (pts (xy 128.045068 61.975583) (xy 128.131861 61.827289) (xy 128.210816 61.673747) (xy 128.306253 61.530366))
     (stroke (width 0.35) (type solid)) (layer "Edge.Cuts"))
+  (gr_text "GLITCHER" (at 155.5 89.65 90) (layer "B.SilkS")
+    (effects (font (size 1 1) (thickness 0.15)) (justify left bottom mirror))
+  )
+  (gr_text "ADC ->" (at 126.2 90.55 -90) (layer "B.SilkS")
+    (effects (font (size 1 1) (thickness 0.15)) (justify left bottom mirror))
+  )
   (gr_text "INPUT" (at 155.3 59.7) (layer "B.SilkS")
     (effects (font (size 2 2) (thickness 0.3)) (justify left bottom mirror))

Commit message: Updated text
Other:
- board text added: "GND"
Changed lines of the file:
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@@
     )
   )
+  (gr_line (start 131.35 85.05) (end 131.575 84.825)
+    (stroke (width 0.15) (type default)) (layer "B.SilkS"))
   (gr_line (start 140.5 75.6) (end 129.9 75.6)
     (stroke (width 0.15) (type default)) (layer "B.SilkS"))
+  (gr_line (start 131.35 81.975) (end 131.575 82.2)
+    (stroke (width 0.15) (type default)) (layer "B.SilkS"))
   (gr_line (start 140.5 60.8) (end 140.5 56.3)
     (stroke (width 0.15) (type default)) (layer "B.SilkS"))
   (gr_line (start 140.5 60.8) (end 140.5 75.6)
+    (stroke (width 0.15) (type default)) (layer "B.SilkS"))
+  (gr_line (start 131.35 81.975) (end 131.125 82.2)
+    (stroke (width 0.15) (type default)) (layer "B.SilkS"))
+  (gr_line (start 131.35 83.45) (end 131.675 83.45)
+    (stroke (width 0.15) (type default)) (layer "B.SilkS"))
+  (gr_line (start 131.35 81.975) (end 131.35 85.05)
+    (stroke (width 0.15) (type default)) (layer "B.SilkS"))
+  (gr_line (start 131.35 85.05) (end 131.125 84.825)
     (stroke (width 0.15) (type default)) (layer "B.SilkS"))
   (gr_curve (pts (xy 140.469802 125.71918) (xy 140.339432 125.693883) (xy 140.207776 125.670058) (xy 140.077879 125.64362))
@@
     (effects (font (size 1 1) (thickness 0.15)) (justify left bottom mirror))
   )
+  (gr_text "GND\n" (at 133.025 81.975 90) (layer "B.SilkS")
+    (effects (font (size 1 1) (thickness 0.15)) (justify left bottom mirror))
+  )

Commit message: Small layout changes
Parts:
- removed D4: LED, LED_SMD:LED_0805_2012Metric
- removed R15, R16: 470, Resistor_SMD:R_0603_1608Metric
- added R9: 470, Resistor_SMD:R_0603_1608Metric, B.Cu at (132.0, 107.4)
- D1, D2, D3: moved to B.Cu
- Q1: value DMN3300U -> AO3400
- moved D3 10.3 mm to (132.2, 104.0), turned to -90 degrees
- moved D2 8.60 mm to (130.2, 104.0), turned to -90 degrees
- moved D1 7.60 mm to (128.2, 104.0), turned to -90 degrees
- moved R14 4.88 mm to (130.2, 107.4), turned to -90 degrees
- moved R13 3.86 mm to (128.5, 107.4), turned to -90 degrees
- moved C13 0.30 mm to (153.0, 99.1)
- moved C12 0.28 mm to (153.0, 97.6)
Connections:
- U1 pad 17: Net-(U1-GPIO14) -> unconnected-(U1-GPIO14-Pad17)
Routing:
- net Net-(U1-GPIO14): track 23.0 -> 0.00 mm
- net Net-(U1-GPIO15): track 25.3 -> 14.8 mm
- net Net-(U1-GPIO13): track 21.1 -> 17.1 mm
- net Net-(D4-A): track 2.66 -> 0.00 mm, vias 1 -> 0
- net Net-(U1-GPIO12): track 18.2 -> 19.2 mm
- net +5V: track 82.4 -> 81.6 mm
- net Net-(D3-A): track 2.45 -> 1.74 mm, vias 1 -> 0
- net Net-(D1-A): track 2.43 -> 1.74 mm, vias 1 -> 0
- net Net-(D2-A): track 2.25 -> 1.64 mm, vias 1 -> 0
- net GND: track 144.2 -> 143.8 mm, vias 38 -> 37
Other:
- board text added: "<- ADC"
- board text added: "ARM"
- board text added: "JW"
- board text added: "TRIG"
- board text added: "USB"
- board text removed: "ADC ->"

Commit message: Prod hw
Parts:
- D1: value LED -> LED RED
- D2, D3: value LED -> LED YELLOW
Routing:
- net +5V: track 81.6 -> 79.9 mm
Other:
- board text added: "Art by ankhaneko.art"
- board text added: "BOLT"
- board text added: "Glitching multitool by curious.supplies"
- board text added: "OUTPUT"
- board text removed: "OUT"
