File: glitcher/glitcher.kicad_sch (KiCad schematic)
At the start: 79 parts, among them J1 USB_C_Receptacle_USB2.0, J2 Conn_01x02, J3 IN, J4 OUT, J5 Conn_01x02, Q1 DMN3300U, SW3 SW_Push, U1 RP2040, U3 W25Q128JVS, U5 AMS1117-3.3, U5 COS722SR, U6 MS9280, Y1 12MHz

Commit message: Routed glitcher
Parts:
- removed J2: Conn_01x02, Connector_PinHeader_2.54mm:PinHeader_1x02_P2.54mm_Horizontal, symbol Connector_Generic:Conn_01x02
- removed J3: IN, Connector_PinHeader_2.54mm:PinHeader_1x08_P2.54mm_Vertical, symbol Connector_Generic:Conn_01x08
- removed J4: OUT, Connector_PinHeader_2.54mm:PinHeader_1x04_P2.54mm_Vertical, symbol Connector_Generic:Conn_01x04
- removed J5: Conn_01x02, Connector_PinHeader_2.54mm:PinHeader_1x02_P2.54mm_Vertical, symbol Connector_Generic:Conn_01x02
- removed R8, R9: 1k, Resistor_SMD:R_0603_1608Metric, symbol Device:R
- removed SW3 (x2): SW_Push, Button_Switch_SMD:SW_Push_1P1T_NO_6x6mm_H9.5mm, symbol Switch:SW_Push
- removed TP1 (x2): TestPoint, TestPoint:TestPoint_Bridge_Pitch2.54mm_Drill1.3mm, symbol Connector:TestPoint
- added C29: 1uF, Capacitor_SMD:C_0603_1608Metric, symbol Device:C
- added J3, J4, J6: Conn_01x05, Connector_PinHeader_2.54mm:PinHeader_1x05_P2.54mm_Vertical_SMD_Pin1Left, symbol Connector_Generic:Conn_01x05
- added J5, J7: Conn_01x03, Connector_PinHeader_2.54mm:PinHeader_1x03_P2.54mm_Vertical_SMD_Pin1Left, symbol Connector_Generic:Conn_01x03
- added R5 (x2): 5.1k, Resistor_SMD:R_0603_1608Metric, symbol Device:R
- added TP1, TP2: TestPoint, TestPoint:TestPoint_Pad_D2.0mm, symbol Connector:TestPoint
Connections:
- net CLK: now also U1.29 (GPIO18); no longer U1.17 (GPIO14)
- net D0: now also U1.30 (GPIO19); no longer U1.18 (GPIO15)
- net D1: now also U1.31 (GPIO20); no longer U1.27 (GPIO16)
- net D2: now also U1.32 (GPIO21); no longer U1.28 (GPIO17)
- net D3: now also U1.34 (GPIO22); no longer U1.29 (GPIO18)
- net D4: now also U1.35 (GPIO23); no longer U1.30 (GPIO19)
- net D5: now also U1.36 (GPIO24); no longer U1.31 (GPIO20)
- net D6: now also U1.37 (GPIO25); no longer U1.32 (GPIO21)
- net D7: now also U1.38 (GPIO26_ADC0); no longer U1.34 (GPIO22)
- net D8: now also U1.39 (GPIO27_ADC1); no longer U1.35 (GPIO23)
- net D9: now also U1.40 (GPIO28_ADC2); no longer U1.36 (GPIO24)
- net GND: now also U5.5 (+), U5.6 (-), C29.2, J3.5 (Pin_5), J4.5 (Pin_5), J5.1 (Pin_1), J5.3 (Pin_3), J6.5 (Pin_5), J7.1 (Pin_1), J7.3 (Pin_3), R5.1, TP1.1; no longer U5.3 (+)
- net OTR: now also U1.41 (GPIO29_ADC3); no longer U1.37 (GPIO25)
- net at R19.1: now also J6.2 (Pin_2)
- net at C21.1, C22.1, U6.21 (REFTS)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: now also R5.2
- net at R30.1: now also J4.1 (Pin_1)
- net at R29.1: now also J4.2 (Pin_2)
- net at R28.1: now also J4.3 (Pin_3)
- net at R27.1: now also J4.4 (Pin_4)
- net at R26.1: now also J3.1 (Pin_1)
- net at R25.1: now also J3.2 (Pin_2)
- net at R24.1: now also J3.3 (Pin_3)
- net at R23.1: now also J3.4 (Pin_4)
- net at R18.1: now also J6.3 (Pin_3)
- net at Q1.3 (D): now also J7.2 (Pin_2)
- net at R10.1, U5.1: now also R12.2
- net at U1.15 (GPIO12): now also R12.2
- net at U1.16 (GPIO13): now also R13.2; no longer R21.2
- net at R14.2: now also U1.17 (GPIO14); no longer U1.40 (GPIO28_ADC2)
- net at R15.2: now also U1.18 (GPIO15); no longer U1.41 (GPIO29_ADC3)
- net at R7.2: now also TP2.1
- net at C20.1: now also J5.2 (Pin_2)
- net at R17.1: now also J6.4 (Pin_4)
- net at R20.1: now also J6.1 (Pin_1)
- new net: R21.2, U1.28 (GPIO17)
- new net: C29.1, R5.1, R5.2, U5.3 (+)
- now unconnected: U5.7
- no-connect marks 3 -> 6
Other:
- moved on the sheet: C19, D1, D2, D3, D4, R12, R13, R14, R15, U5C

Commit message: Updated text
Parts:
- J3, J4, J6: LCSC (none) -> C2883802
- J5, J7: LCSC (none) -> C780061
Changed lines of the file:
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@@
+      (effects (font (size 1.27 1.27)) hide)
+    )
+    (property "LCSC" "C2883802" (at 201.93 57.15 0)
       (effects (font (size 1.27 1.27)) hide)
     )
@@
       (effects (font (size 1.27 1.27)) hide)
     )
+    (property "LCSC" "C2883802" (at 191.77 67.31 0)
+      (effects (font (size 1.27 1.27)) hide)
+    )
     (pin "1")
     (pin "2")
@@
       (effects (font (size 1.27 1.27)) hide)
     )
+    (property "LCSC" "C780061" (at 19.05 153.67 0)
+      (effects (font (size 1.27 1.27)) hide)
+    )
     (pin "1")
     (pin "2")
@@
       (effects (font (size 1.27 1.27)) hide)
     )
+    (property "LCSC" "C2883802" (at 181.61 77.47 0)
+      (effects (font (size 1.27 1.27)) hide)
+    )
     (pin "1")
     (pin "2")
@@
       (effects (font (size 1.27 1.27)) hide)
     )
+    (property "LCSC" "C780061" (at 215.9 92.71 0)
+      (effects (font (size 1.27 1.27)) hide)
+    )

Commit message: Small layout changes
Parts:
- removed D3, D4: LED, LED_SMD:LED_0805_2012Metric, symbol Device:LED
- removed R14, R15: 470, Resistor_SMD:R_0603_1608Metric, symbol Device:R
- added D2: LED, LED_SMD:LED_0805_2012Metric, symbol Device:LED
- added R13: 470, Resistor_SMD:R_0603_1608Metric, symbol Device:R
- Q1: value DMN3300U -> AO3400; LCSC C461018 -> C20917
- R6: now not fitted
Connections:
- net GND: now also D2.1 (K)
- net at U1.18 (GPIO15): now also R13.2
- new net: D2.2 (A), R13.1

Commit message: Prod hw
Parts:
- D1: value LED -> LED RED
- D2: value LED -> LED YELLOW
- J3, J4, J6: LCSC C2883802 -> C5160788
- J5, J7: LCSC C780061 -> C5160786
Changed lines of the file:
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@@
       (effects (font (size 1.27 1.27)) hide)
     )
-    (property "LCSC" "C2883802" (at 201.93 57.15 0)
+    (property "LCSC" "C5160788" (at 201.93 57.15 0)
       (effects (font (size 1.27 1.27)) hide)
     )
@@
       (effects (font (size 1.27 1.27)))
     )
-    (property "Value" "LED" (at 186.69 125.73 0)
+    (property "Value" "LED RED" (at 186.69 125.73 0)
       (effects (font (size 1.27 1.27)) hide)
     )
@@
       (effects (font (size 1.27 1.27)))
     )
-    (property "Value" "LED" (at 181.61 125.73 0)
+    (property "Value" "LED YELLOW" (at 181.61 125.73 0)
       (effects (font (size 1.27 1.27)) hide)
     )
@@
       (effects (font (size 1.27 1.27)))
     )
-    (property "Value" "LED" (at 184.15 125.73 0)
+    (property "Value" "LED YELLOW" (at 184.15 125.73 0)
       (effects (font (size 1.27 1.27)) hide)
     )
@@
       (effects (font (size 1.27 1.27)) hide)
     )
-    (property "LCSC" "C2883802" (at 191.77 67.31 0)
+    (property "LCSC" "C5160788" (at 191.77 67.31 0)
       (effects (font (size 1.27 1.27)) hide)
     )
@@
       (effects (font (size 1.27 1.27)) hide)
     )
-    (property "LCSC" "C780061" (at 19.05 153.67 0)
+    (property "LCSC" "C5160786" (at 19.05 153.67 0)
       (effects (font (size 1.27 1.27)) hide)
     )
@@
       (effects (font (size 1.27 1.27)) hide)
     )
-    (property "LCSC" "C2883802" (at 181.61 77.47 0)
+    (property "LCSC" "C5160788" (at 181.61 77.47 0)
       (effects (font (size 1.27 1.27)) hide)
     )
@@
       (effects (font (size 1.27 1.27)) hide)
     )
-    (property "LCSC" "C780061" (at 215.9 92.71 0)
-      (effects (font (size 1.27 1.27)) hide)
-    )
+    (property "LCSC" "C5160786" (at 215.9 92.71 0)
+      (effects (font (size 1.27 1.27)) hide)
+    )
